Commit message: some collisions and delete complex mishes

File: urdf/antares.urdf (robot description, URDF)
Before this commit: robot antares, 21 links, 20 joints
Links:
- link base_link: geometry collision box size=0,23 0,115 0,235; visual mesh filename=package://antares_model/meshes/body_visual_simple.stl
- link head: geometry collision box size=0,07 0,12 0,037; visual mesh filename=package://antares_model/meshes/head_visual_simple.stl
- link hip_l: geometry collision box size=0,05 0,044 0,21; visual mesh filename=package://antares_model/meshes/hip_l_visual.stl
- link hip_r: geometry collision box size=0,05 0,044 0,21; visual mesh filename=package://antares_model/meshes/hip_r_visual.stl
- link neck: geometry collision box size=0,034 0,035 0,07; visual mesh filename=package://antares_model/meshes/neck_visual_simple.stl
- link pelvis_l: geometry collision box size=0,053 0,064 0,04; visual mesh filename=package://antares_model/meshes/pelvis_l_visual_simple.stl
- link pelvis_l_servos: geometry collision box size=0,039 0,105 0,062; visual mesh filename=package://antares_model/meshes/pelvis_servos_l_visual_simpl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
- link pelvis_r: geometry collision box size=0,053 0,064 0,04; visual mesh filename=package://antares_model/meshes/pelvis_r_visual_simple.stl
- link pelvis_r_servos: geometry collision box size=0,039 0,105 0,062; visual mesh filename=package://antares_model/meshes/pelvis_servos_r_visual_simpl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

Commit message: more simple meshes and collision primitives

File: urdf/antares.urdf (robot description, URDF)
Before this commit: robot antares, 21 links, 20 joints
Links:
- link ankle_l: geometry collision box size=0,105 0,2 0,01; visual mesh filename=package://antares_model/meshes/ankle_l_visual_simple.stl
- link ankle_l_servos: geometry collision box size=0,045 0,1 0,06; visual mesh filename=package://antares_model/meshes/ankle_l_servos_visual_simple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
- link ankle_r: geometry collision box size=0,105 0,2 0,01; visual mesh filename=package://antares_model/meshes/ankle_r_visual_simple.stl
- link ankle_r_servos: geometry collision box size=0,045 0,1 0,06; visual mesh filename=package://antares_model/meshes/ankle_r_servos_visual_simple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
- link calf_l: geometry collision box size=0,087 0,04 0,19; visual mesh filename=package://antares_model/meshes/calf_l_visual_simple.stl
- link calf_r: geometry collision box size=0,087 0,04 0,19; visual mesh filename=package://antares_model/meshes/calf_r_visual_simple.stl
- link hip_l: geometry collision box size=0,05 0,044 0,21; visual mesh filename=package://antares_model/meshes/hip_l_visual_simple.stl
- link hip_r: geometry collision box size=0,05 0,044 0,21; visual mesh filename=package://antares_model/meshes/hip_r_visual_simple.stl

Commit message: all meshes are replaced with simplified versions

File: urdf/antares.urdf (robot description, URDF)
Before this commit: robot antares, 21 links, 20 joints
Links:
- link forearm_l: geometry visual mesh filename=package://antares_model/meshes/forearm_l_visual_simple.stl
- link forearm_r: geometry visual mesh filename=package://antares_model/meshes/forearm_r_visual_simple.stl
- link lower_shoulder_l: geometry visual mesh filename=package://antares_model/meshes/lower_shoulder_l_visual_simp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
- link lower_shoulder_r: geometry visual mesh filename=package://antares_model/meshes/lower_shoulder_r_visual_simp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
- link shoulder_l: geometry visual mesh filename=package://antares_model/meshes/upper_shoulder_l_visual_simp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
- link shoulder_r: geometry visual mesh filename=package://antares_model/meshes/upper_shoulder_r_visual_simp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

Commit message: collisions primitives added to all links

File: urdf/antares.urdf (robot description, URDF)
Before this commit: robot antares, 21 links, 20 joints
Links:
- link forearm_l: geometry collision box size=0,03 0,0465 0,16; visual mesh filename=package://antares_model/meshes/forearm_l_visual_simple.stl
- link forearm_r: geometry collision box size=0,03 0,0465 0,16; visual mesh filename=package://antares_model/meshes/forearm_r_visual_simple.stl
- link lower_shoulder_l: geometry collision box size=0,036 0,036 0,17; visual mesh filename=package://antares_model/meshes/lower_shoulder_l_visual_simp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
- link lower_shoulder_r: geometry collision box size=0,036 0,036 0,17; visual mesh filename=package://antares_model/meshes/lower_shoulder_r_visual_simp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
- link shoulder_l: geometry collision box size=0,04 0,044 0,03; visual mesh filename=package://antares_model/meshes/upper_shoulder_l_visual_simp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
- link shoulder_r: geometry collision box size=0,04 0,044 0,03; visual mesh filename=package://antares_model/meshes/upper_shoulder_r_visual_simp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
Joints:
- removed joint ankle_l_servos_to_ankle
- removed joint ankle_r_servos_to_ankle
- removed joint body_to_neck
- removed joint body_to_pelvis_l
- removed joint body_to_pelvis_r
- removed joint body_to_shoulder_l
- removed joint body_to_shoulder_r
- removed joint calf_l_to_ankle_servos
- removed joint calf_r_to_ankle_servos
- removed joint hip_l_to_calf
- removed joint hip_r_to_calf
- removed joint lower_shoulder_l_to_forearm
- removed joint lower_shoulder_r_to_forearm
- removed joint neck_to_head
- removed joint pelvis_l_servos_to_hip
- removed joint pelvis_l_to_pelvis_servos
- removed joint pelvis_r_servos_to_hip
- removed joint pelvis_r_to_pelvis_servos
- removed joint shoulder_to_lower_shoulder_l
- removed joint shoulder_to_lower_shoulder_r
- added joint ankle_pitch_l: type continuous, parent calf_l, child ankle_l_servos, origin xyz=0 0.003 -0.170075 rpy=0 0 0, axis 1 0 0
- added joint ankle_pitch_r: type continuous, parent calf_r, child ankle_r_servos, origin xyz=0 0.003 -0.170075 rpy=0 0 0, axis 1 0 0
- added joint ankle_roll_l: type continuous, parent ankle_l_servos, child ankle_l, origin xyz=0 0 0 rpy=0 0 0, axis 0 1 0
- added joint ankle_roll_r: type continuous, parent ankle_r_servos, child ankle_r, origin xyz=0 0 0 rpy=0 0 0, axis 0 1 0
- added joint elbow_pitch_l: type continuous, parent lower_shoulder_l, child forearm_l, origin xyz=0 0 -0.14048 rpy=0 0 0, axis 1 0 0
- added joint elbow_pitch_r: type continuous, parent lower_shoulder_r, child forearm_r, origin xyz=0 0 -0.14048 rpy=0 0 0, axis 1 0 0
- added joint head_pitch: type continuous, parent neck, child head, origin xyz=0 0 0.022976 rpy=0 0 0, axis 1 0 0
- added joint head_yaw: type continuous, parent base_link, child neck, origin xyz=0.17762 -0.086853 0.72319 rpy=0 0 0, axis 0 0 1
- added joint knee_pitch_l: type continuous, parent hip_l, child calf_l, origin xyz=0 0.001 -0.1759 rpy=0 0 0, axis 1 0 0
- added joint knee_pitch_r: type continuous, parent hip_r, child calf_r, origin xyz=0 0.001 -0.1759 rpy=0 0 0, axis 1 0 0
- added joint pelvis_pitch_l: type continuous, parent pelvis_l_servos, child hip_l, origin xyz=0 0 0 rpy=0 0 0, axis 1 0 0
- added joint pelvis_pitch_r: type continuous, parent pelvis_r_servos, child hip_r, origin xyz=0 0 0 rpy=0 0 0, axis 1 0 0
- added joint pelvis_roll_l: type continuous, parent pelvis_l, child pelvis_l_servos, origin xyz=-0.00017 0 -0.01252 rpy=0 0 0, axis 0 1 0
- added joint pelvis_roll_r: type continuous, parent pelvis_r, child pelvis_r_servos, origin xyz=0.00017 0 -0.01252 rpy=0 0 0, axis 0 1 0
- added joint pelvis_yaw_l: type continuous, parent base_link, child pelvis_l, origin xyz=0.26206 -0.099753 0.43020 rpy=0 0 0, axis 0 0 1
- added joint pelvis_yaw_r: type continuous, parent base_link, child pelvis_r, origin xyz=0.093392 -0.099753 0.43020 rpy=0 0 0, axis 0 0 1
- added joint shoulder_pitch_l: type continuous, parent base_link, child shoulder_l, origin xyz=0.29596 -0.099723 0.64948 rpy=0 0 0, axis 1 0 0
- added joint shoulder_pitch_r: type continuous, parent base_link, child shoulder_r, origin xyz=0.059497 -0.099723 0.64948 rpy=0 0 0, axis 1 0 0
- added joint shoulder_roll_l: type continuous, parent shoulder_l, child lower_shoulder_l, origin xyz=0.03287 -0.00003 0.00003 rpy=0 0 0, axis 0 1 0
- added joint shoulder_roll_r: type continuous, parent shoulder_r, child lower_shoulder_r, origin xyz=-0.03287 -0.00003 0.00003 rpy=0 0 0, axis 0 1 0

Commit message: fix elbow joint names, add launch files

File: urdf/antares.urdf (robot description, URDF)
Before this commit: robot antares, 21 links, 20 joints
Joints:
- removed joint elbow_pitch_l
- removed joint elbow_pitch_r
- added joint elbow_l: type continuous, parent lower_shoulder_l, child forearm_l, origin xyz=0 0 -0.14048 rpy=0 0 0, axis 1 0 0
- added joint elbow_r: type continuous, parent lower_shoulder_r, child forearm_r, origin xyz=0 0 -0.14048 rpy=0 0 0, axis 1 0 0
